Commit message: Tweaks in URDF and remove unneeded t265 frame

File: o_description/urdf/o.urdf.xacro (robot description, xacro)
@@ -102,8 +102,8 @@
   </xacro:wheel>
   <xacro:caster wheel_prefix="lcaster">
-    <origin xyz="${fwheel_offset} 0.135 ${-caster_radius}" rpy="0 0 0" />
+    <origin xyz="${fwheel_offset} 0.135 -0.086" rpy="0 0 0" />
   </xacro:caster>
   <xacro:caster wheel_prefix="rcaster">
-    <origin xyz="${fwheel_offset} -0.135 ${-caster_radius}" rpy="0 0 0" />
+    <origin xyz="${fwheel_offset} -0.135 -0.086" rpy="0 0 0" />
   </xacro:caster>
   <link name="neato">
@@ -168,5 +168,5 @@
     <parent link="base_link" />
     <child link="t265_camera_link" />
-    <origin xyz="${stereo_plate_x_offset} 0 ${stereo_plate_z_offset-0.030}" rpy="0 0 0" />
+    <origin xyz="0.135 0 0.235" rpy="0 0 0" />
   </joint>
 </robot>

Commit message: Changes for new camera plate

File: o_description/urdf/o.urdf.xacro (robot description, xacro)
@@ -39,5 +39,5 @@
   <xacro:property name="wheel_offset_from_front" value="0.129" />
   <xacro:property name="stereo_plate_x_offset" value="0.160" />
-  <xacro:property name="stereo_plate_z_offset" value="${0.258+0.0124}" />
+  <xacro:property name="stereo_plate_z_offset" value="${0.241}" />
   <xacro:property name="d435_y_offset" value="0.077" />
   <xacro:property name="lidar_x_offset" value="-0.130" />
@@ -181,5 +181,5 @@
     <parent link="base_link" />
     <child link="t265_camera_link" />
-    <origin xyz="${0.165-(t265_width/2)} 0 ${0.229+(t265_height/2)}" rpy="0 0 0" />
+    <origin xyz="${0.165} 0 ${0.275}" rpy="0 0.1388 0" />
   </joint>
 </robot>

Commit message: launch file fix and angle fix for t265 for new stereo camera plate

File: o_description/urdf/o.urdf.xacro (robot description, xacro)
@@ -181,5 +181,5 @@
     <parent link="base_link" />
     <child link="t265_camera_link" />
-    <origin xyz="${0.165} 0 ${0.275}" rpy="0 0.1388 0" />
+    <origin xyz="${0.165} 0 ${-0.275}" rpy="0 0.1388 0" />
   </joint>
 </robot>

Commit message: Snapshot trying to get laser merge to work and frames correct

File: o_description/urdf/o.urdf.xacro (robot description, xacro)
@@ -181,5 +181,5 @@
     <parent link="base_link" />
     <child link="t265_camera_link" />
-    <origin xyz="${0.165} 0 ${-0.275}" rpy="0 0.1388 0" />
+    <origin xyz="${0.165} 0 ${0.275}" rpy="0 -0.1388 0" />
   </joint>
 </robot>
